Commit message: Add and configure IMU sensor for Gazebo

File: install/robotpadi/share/robotpadi/urdf/imu.xacro (robot description, xacro)
@@ -34,8 +34,8 @@
         <visualize>true</visualize>
         <topic>imu/data</topic>
-        <plugin filename="libgz_ros2_imu_bridge.so" name="imu_bridge_plugin">
+        <!-- <plugin filename="libgz_ros2_imu_bridge.so" name="imu_bridge_plugin">
           <ros_topic>imu/data</ros_topic>
           <frame_id>${imu_link_name}</frame_id>
-        </plugin>
+        </plugin> -->
       </sensor>
     </gazebo>

File: robotpadi/urdf/imu.xacro (robot description, xacro)
@@ -7,6 +7,6 @@
         <geometry>
           <box size="0.1 0.1 0.1"/> </geometry>
-        <material name="blue">
-          <color rgba="0 0 1 1"/>
+        <material name="black">
+          <color rgba="0 0 0 1"/>
         </material>
       </visual>
@@ -34,8 +34,8 @@
         <visualize>true</visualize>
         <topic>imu/data</topic>
-        <plugin filename="libgz_ros2_imu_bridge.so" name="imu_bridge_plugin">
+        <!-- <plugin filename="libgz_ros2_imu_bridge.so" name="imu_bridge_plugin">
           <ros_topic>imu/data</ros_topic>
           <frame_id>${imu_link_name}</frame_id>
-        </plugin>
+        </plugin> -->
       </sensor>
     </gazebo>

Commit message: teleop gazebo rviz sync, imu pembacaan quaternion

File: install/robotpadi/share/robotpadi/urdf/imu.xacro (robot description, xacro)
@@ -7,6 +7,6 @@
         <geometry>
           <box size="0.1 0.1 0.1"/> </geometry>
-        <material name="blue">
-          <color rgba="0 0 1 1"/>
+        <material name="black">
+          <color rgba="0 0 0 1"/>
         </material>
       </visual>
@@ -38,4 +38,49 @@
           <frame_id>${imu_link_name}</frame_id>
         </plugin> -->
+        <plugin filename="libignition-gazebo-imu-system.so"
+        name="ignition::gazebo::systems::Imu">
+        </plugin>
+      <!-- <imu>
+        <angular_velocity>
+          <x>
+            <noise type="gaussian">
+              <mean>0.0</mean>
+              <stddev>2e-4</stddev>
+            </noise>
+          </x>
+          <y>
+            <noise type="gaussian">
+              <mean>0.0</mean>
+              <stddev>2e-4</stddev>
+            </noise>
+          </y>
+          <z>
+            <noise type="gaussian">
+              <mean>0.0</mean>
+              <stddev>2e-4</stddev>
+            </noise>
+          </z>
+        </angular_velocity>
+        <linear_acceleration>
+          <x>
+            <noise type="gaussian">
+              <mean>0.0</mean>
+              <stddev>1.7e-2</stddev>
+            </noise>
+          </x>
+          <y>
+            <noise type="gaussian">
+              <mean>0.0</mean>
+              <stddev>1.7e-2</stddev>
+            </noise>
+          </y>
+          <z>
+            <noise type="gaussian">
+              <mean>0.0</mean>
+              <stddev>1.7e-2</stddev>
+            </noise>
+          </z>
+        </linear_acceleration>
+      </imu> -->
       </sensor>
     </gazebo>

File: install/robotpadi/share/robotpadi/urdf/robot_padi.xacro (robot description, xacro)
@@ -201,5 +201,5 @@
       link="Wheel_FR_Link" />
     <axis
-      xyz="0 -1 0" />
+      xyz="0 1 0" />
   </joint>
   <link
@@ -252,5 +252,5 @@
       link="Wheel_RR_Link" />
     <axis
-      xyz="0 -1 0" />
+      xyz="0 1 0" />
   </joint>
   <gazebo reference="base_link">

File: robotpadi/urdf/imu.xacro (robot description, xacro)
@@ -38,4 +38,49 @@
           <frame_id>${imu_link_name}</frame_id>
         </plugin> -->
+        <plugin filename="libignition-gazebo-imu-system.so"
+        name="ignition::gazebo::systems::Imu">
+        </plugin>
+      <!-- <imu>
+        <angular_velocity>
+          <x>
+            <noise type="gaussian">
+              <mean>0.0</mean>
+              <stddev>2e-4</stddev>
+            </noise>
+          </x>
+          <y>
+            <noise type="gaussian">
+              <mean>0.0</mean>
+              <stddev>2e-4</stddev>
+            </noise>
+          </y>
+          <z>
+            <noise type="gaussian">
+              <mean>0.0</mean>
+              <stddev>2e-4</stddev>
+            </noise>
+          </z>
+        </angular_velocity>
+        <linear_acceleration>
+          <x>
+            <noise type="gaussian">
+              <mean>0.0</mean>
+              <stddev>1.7e-2</stddev>
+            </noise>
+          </x>
+          <y>
+            <noise type="gaussian">
+              <mean>0.0</mean>
+              <stddev>1.7e-2</stddev>
+            </noise>
+          </y>
+          <z>
+            <noise type="gaussian">
+              <mean>0.0</mean>
+              <stddev>1.7e-2</stddev>
+            </noise>
+          </z>
+        </linear_acceleration>
+      </imu> -->
       </sensor>
     </gazebo>
