Commit message: teleop key bener

File: install/robotpadi/share/robotpadi/urdf/robot_padi.xacro (robot description, xacro)
@@ -19,5 +19,5 @@
       <mass
         value="180" />
-      <inertia
+      <!-- <inertia
         ixx="2.32881913674761"
         ixy="3.13125017353562E-06"
@@ -25,5 +25,12 @@
         iyy="1.87881391838459"
         iyz="-1.67327823321756E-07"
-        izz="2.97314088623897" />
+        izz="2.97314088623897" /> -->
+      <inertia
+        ixx="25.4"
+        ixy="0"
+        ixz="0"
+        iyy="35.1"
+        iyz="0"
+        izz="38.2" />
     </inertial>
     <visual>
@@ -49,5 +56,5 @@
     </collision>
   </link>
-   <xacro:imu_sensor parent_link="base_link" imu_link_name="imu_link" origin_xyz="0.1 0 0.05" origin_rpy="0 0 0"/>
+   <xacro:imu_sensor parent_link="base_link" imu_link_name="imu_link" origin_xyz="0 0 0.05" origin_rpy="0 0 0"/>
   <link
     name="Wheel_FL_Link">

File: install/robotpadi/share/robotpadi/urdf/ros2_control.xacro (robot description, xacro)
@@ -28,5 +28,5 @@
    <gazebo>
       <plugin filename="gz_ros2_control-system" name="gz_ros2_control::GazeboSimROS2ControlPlugin">
-        <parameters>/home/satyo03/TA/install/robotpadi/share/robotpadi/config/diff_drive_controller.yaml</parameters>
+        <parameters>/home/satyo03/TA_robotpadi/install/robotpadi/share/robotpadi/config/diff_drive_controller.yaml</parameters>
       </plugin>
   </gazebo>
