Commit message: robot berjalan tapi random

File: install/robotpadi/share/robotpadi/urdf/gazebo_plugin.xacro (robot description, xacro)
@@ -1 +1,22 @@
-/home/satyo03/TA_robotpadi/robotpadi/urdf/gazebo_plugin.xacro
+<?xml version="1.0"?>
+<robot xmlns:xacro="http://ros.org/wiki/xacro">
+  <xacro:arg name="namespace" default="" />
+  <!-- <gazebo>
+    <plugin filename="libignition-gazebo-sensors-system.so"
+      name="ignition::gazebo::systems::Sensors">
+      <render_engine>ogre2</render_engine>
+    </plugin>
+    <plugin name="ignition::gazebo::systems::Imu" filename="libignition-gazebo-imu-system.so" />
+    <plugin filename="ign_ros2_control-system" name="ign_ros2_control::IgnitionROS2ControlPlugin">
+      <parameters>$(find robotpadi)/config/diff_drive_controller.yaml</parameters>
+    </plugin>
+  </gazebo> -->
+  <gazebo>
+      <plugin filename="gz_ros2_control-system" name="gz_ros2_control::GazeboSimROS2ControlPlugin">
+      <ros>
+          <namespace>$(arg namespace)</namespace>
+      </ros>
+      <parameters>$(find robotpadi)/config/diff_drive_controller.yaml</parameters>
+      </plugin>
+  </gazebo>
+</robot>

File: install/robotpadi/share/robotpadi/urdf/imu.xacro (robot description, xacro)
@@ -1 +1,151 @@
-/home/satyo03/TA_robotpadi/robotpadi/urdf/imu.xacro
+<?xml version="1.0"?>
+<robot xmlns:xacro="http://www.ros.org/wiki/xacro">
+  <xacro:macro name="imu_sensor" params="parent_link imu_link_name origin_xyz origin_rpy">
+    <link name="${imu_link_name}">
+      <visual>
+        <origin xyz="0 0 0" rpy="0 0 0"/>
+        <geometry>
+          <box size="0.1 0.1 0.1"/> </geometry>
+        <material name="black">
+          <color rgba="0 0 0 1"/>
+        </material>
+      </visual>
+      <collision>
+        <origin xyz="0 0 0" rpy="0 0 0"/>
+        <geometry>
+          <box size="0.1 0.1 0.1"/>
+        </geometry>
+      </collision>
+      <inertial>
+        <origin xyz="0 0 0" rpy="0 0 0"/>
+        <mass value="0.01"/>
+        <inertia ixx="0.000001" ixy="0" ixz="0" iyy="0.000001" iyz="0" izz="0.000001"/>
+      </inertial>
+    </link>
+    <joint name="${imu_link_name}_joint" type="fixed">
+      <parent link="${parent_link}"/>
+      <child link="${imu_link_name}"/>
+      <origin xyz="${origin_xyz}" rpy="${origin_rpy}"/>
+    </joint>
+    <gazebo reference="${imu_link_name}">
+      <sensor name="imu_sensor" type="imu">
+        <always_on>true</always_on>
+        <update_rate>100</update_rate>
+        <visualize>true</visualize>
+        <topic>imu/data</topic>
+        <!-- <plugin filename="libgz_ros2_imu_bridge.so" name="imu_bridge_plugin">
+          <ros_topic>imu/data</ros_topic>
+          <frame_id>${imu_link_name}</frame_id>
+        </plugin> -->
+        <plugin filename="libgazebo_ros_imu_sensor.so" name="imu_plugin">
+          <ros>
+            <namespace>/</namespace>
+            <topic>/imu/data</topic>
+          </ros>
+          <initial_orientation_as_reference>false</initial_orientation_as_reference>
+        </plugin>
+      <!-- <imu>
+        <angular_velocity>
+          <x>
+            <noise type="gaussian">
+              <mean>0.0</mean>
+              <stddev>2e-4</stddev>
+            </noise>
+          </x>
+          <y>
+            <noise type="gaussian">
+              <mean>0.0</mean>
+              <stddev>2e-4</stddev>
+            </noise>
+          </y>
+          <z>
+            <noise type="gaussian">
+              <mean>0.0</mean>
+              <stddev>2e-4</stddev>
+            </noise>
+          </z>
+        </angular_velocity>
+        <linear_acceleration>
+          <x>
+            <noise type="gaussian">
+              <mean>0.0</mean>
+              <stddev>1.7e-2</stddev>
+            </noise>
+          </x>
+          <y>
+            <noise type="gaussian">
+              <mean>0.0</mean>
+              <stddev>1.7e-2</stddev>
+            </noise>
+          </y>
+          <z>
+            <noise type="gaussian">
+              <mean>0.0</mean>
+              <stddev>1.7e-2</stddev>
+            </noise>
+          </z>
+        </linear_acceleration>
+      </imu> -->
+      </sensor>
+    </gazebo>
+  </xacro:macro>
+</robot>
+<!-- <?xml version="1.0"?>
+<robot xmlns:xacro="http://www.ros.org/wiki/xacro">
+  <xacro:macro name="imu_sensor" params="parent_link imu_link_name origin_xyz origin_rpy">
+    <link name="${imu_link_name}">
+      <visual>
+        <origin xyz="0 0 0" rpy="0 0 0"/>
+        <geometry>
+          <box size="0.01 0.01 0.01"/> </geometry>
+        <material name="black">
+          <color rgba="0 0 0 1"/>
+        </material>
+      </visual>
+      <collision>
+        <origin xyz="0 0 0" rpy="0 0 0"/>
+        <geometry>
+          <box size="0.01 0.01 0.01"/>
+        </geometry>
+      </collision>
+      <inertial>
+        <origin xyz="0 0 0" rpy="0 0 0"/>
+        <mass value="0.01"/>
+        <inertia ixx="0.000001" ixy="0" ixz="0" iyy="0.000001" iyz="0" izz="0.000001"/>
+      </inertial>
+    </link>
+    <joint name="${imu_link_name}_joint" type="fixed">
+      <parent link="${parent_link}"/>
+      <child link="${imu_link_name}"/>
+      <origin xyz="${origin_xyz}" rpy="${origin_rpy}"/>
+    </joint> -->
+<!-- batas -->
+    <!-- <gazebo reference="${imu_link_name}">
+      <plugin filename="libgazebo_ros_imu_sensor.so" name="imu_sensor_plugin">
+        <ros>
+          <namespace>/</namespace>
+          <remapping>imu:imu/data</remapping>
+        </ros>
+        <initialOrientationAsReference>false</initialOrientationAsReference>
+        <updateRate>100.0</updateRate>
+        <gaussianNoise>0.005</gaussianNoise>
+        <topicName>imu/data</topicName>
+        <frameName>${imu_link_name}</frameName>
+      </plugin>
+    </gazebo> -->
+<!-- batas -->
+    <!-- <gazebo>
+      <plugin filename="libgazebo_ros_imu_sensor.so" name="imu_sensor_plugin">
+        <ros>
+          <namespace>/</namespace>
+          <remapping>imu:imu/data</remapping>
+        </ros>
+        <initialOrientationAsReference>false</initialOrientationAsReference>
+        <updateRate>100.0</updateRate>
+        <gaussianNoise>0.005</gaussianNoise>
+        <topicName>imu/data</topicName>
+        <frameName>${imu_link_name}</frameName>
+      </plugin>
+    </gazebo>
+  </xacro:macro>
+</robot> -->

File: install/robotpadi/share/robotpadi/urdf/main.xacro (robot description, xacro)
@@ -1 +1,6 @@
-/home/satyo03/TA_robotpadi/robotpadi/urdf/main.xacro
+<?xml version="1.0"?>
+<robot xmlns:xacro="http://www.ros.org/wiki/xacro" name="robot_padi">
+    <xacro:include filename="robot_padi.xacro"/>
+    <xacro:include filename="ros2_control.xacro"/>
+    <!-- <xacro:include filename="gazebo_plugin.xacro"/> -->
+</robot>

File: install/robotpadi/share/robotpadi/urdf/robot_padi.xacro (robot description, xacro)
@@ -1 +1,330 @@
-/home/satyo03/TA_robotpadi/robotpadi/urdf/robot_padi.xacro
+<?xml version="1.0" encoding="utf-8"?>
+<!-- This URDF was automatically created by SolidWorks to URDF Exporter! Originally created by Stephen Brawner (brawner@gmail.com)
+     Commit Version: 1.6.0-4-g7f85cfe  Build Version: 1.6.7995.38578
+     For more information, please see http://wiki.ros.org/sw_urdf_exporter -->
+<robot xmlns:xacro="http://www.ros.org/wiki/xacro">
+  <xacro:property name="mesh_path" value="$(find robotpadi)/meshes"/>
+  <xacro:include filename="$(find robotpadi)/urdf/imu.xacro" />
+  <link name="base_footprint"/>
+  <joint name="base_footprint_to_base_link_joint" type="fixed">
+    <parent link="base_footprint"/>
+    <child link="base_link"/>
+  </joint>
+  <link
+    name="base_link">
+    <inertial>
+      <origin
+        xyz="0.0840921680050198 -0.00163983249679742 0.134879064410453"
+        rpy="0 0 0" />
+      <mass
+        value="180" />
+      <!-- <inertia
+        ixx="2.32881913674761"
+        ixy="3.13125017353562E-06"
+        ixz="0.605279043325787"
+        iyy="1.87881391838459"
+        iyz="-1.67327823321756E-07"
+        izz="2.97314088623897" /> -->
+      <inertia
+        ixx="25.4"
+        ixy="0"
+        ixz="0"
+        iyy="35.1"
+        iyz="0"
+        izz="38.2" />
+    </inertial>
+    <visual>
+      <origin
+        xyz="0 0 0"
+        rpy="0 0 0" />
+      <geometry>
+        <mesh filename="file://${mesh_path}/base_link.STL" />
+      </geometry>
+      <material
+        name="">
+        <color
+          rgba="0 0 1 1" />
+      </material>
+    </visual>
+    <collision>
+      <origin
+        xyz="0 0 0"
+        rpy="0 0 0" />
+      <geometry>
+        <mesh filename="file://${mesh_path}/base_link.STL" />
+      </geometry>
+    </collision>
+  </link>
+   <xacro:imu_sensor parent_link="base_link" imu_link_name="imu_link" origin_xyz="0 0 0.05" origin_rpy="0 0 0"/>
+  <link
+    name="Wheel_FL_Link">
+    <inertial>
+      <origin
+        xyz="-1.11022302462516E-16 0.0271089810837371 0"
+        rpy="0 0 0" />
+      <mass
+        value="5" />
+      <inertia
+        ixx="0.00350719044409918"
+        ixy="-9.92501913416296E-14"
+        ixz="4.93198168428617E-17"
+        iyy="0.00624534196811695"
+        iyz="-4.35310172123345E-14"
+        izz="0.00350719044409912" />
+    </inertial>
+    <visual>
+      <origin
+        xyz="0 0 0"
+        rpy="0 0 0" />
+      <geometry>
+        <mesh filename="file://${mesh_path}/Wheel_FL_Link.STL" />
+      </geometry>
+      <material
+        name="">
+        <color
+          rgba="0 0 0 1" />
+      </material>
+    </visual>
+    <collision>
+      <origin
+        xyz="0 0 0"
+        rpy="0 0 0" />
+      <geometry>
+        <mesh filename="file://${mesh_path}/Wheel_FL_Link.STL" />
+      </geometry>
+    </collision>
+  </link>
+  <joint
+    name="Wheel_FL_joint"
+    type="continuous">
+    <origin
+      xyz="0.545 0.437 -0.747"
+      rpy="0 0 0" />
+    <parent
+      link="base_link" />
+    <child
+      link="Wheel_FL_Link" />
+    <axis
+      xyz="0 1 0" />
+  </joint>
+  <!-- transmission -->
+  <transmission name="Wheel_FL_trans">
+    <type>transmission_interface/SimpleTransmission</type>
+    <joint name="Wheel_FL_joint">
+      <hardwareInterface>hardware_interface/VelocityJointInterface</hardwareInterface>
+    </joint>
+    <actuator name="Wheel_FL_motor">
+      <hardwareInterface>hardware_interface/VelocityJointInterface</hardwareInterface>
+      <mechanicalReduction>1</mechanicalReduction>
+    </actuator>
+  </transmission>
+<!-- transmission -->
+  <link
+    name="Wheel_RL_Link">
+    <inertial>
+      <origin
+        xyz="7.7715611723761E-16 0.0241089810837369 6.66133814775094E-16"
+        rpy="0 0 0" />
+      <mass
+        value="5" />
+      <inertia
+        ixx="0.00350719044409904"
+        ixy="9.92519864792002E-14"
+        ixz="-7.45868758339047E-18"
+        iyy="0.0062453419681168"
+        iyz="4.35243565314327E-14"
+        izz="0.00350719044409911" />
+    </inertial>
+    <visual>
+      <origin
+        xyz="0 0 0"
+        rpy="0 0 0" />
+      <geometry>
+        <mesh filename="file://${mesh_path}/Wheel_RL_Link.STL" />
+      </geometry>
+      <material
+        name="">
+        <color
+          rgba="0 0 0 1" />
+      </material>
+    </visual>
+    <collision>
+      <origin
+        xyz="0 0 0"
+        rpy="0 0 0" />
+      <geometry>
+        <mesh filename="file://${mesh_path}/Wheel_RL_Link.STL" />
+      </geometry>
+    </collision>
+  </link>
+  <joint
+    name="Wheel_RL_joint"
+    type="continuous">
+    <origin
+      xyz="-0.545 0.44 -0.747"
+      rpy="0 0 0" />
+    <parent
+      link="base_link" />
+    <child
+      link="Wheel_RL_Link" />
+    <axis
+      xyz="0 1 0" />
+  </joint>
+  <!-- transmission -->
+  <transmission name="Wheel_RL_trans">
+    <type>transmission_interface/SimpleTransmission</type>
+    <joint name="Wheel_RL_joint">
+      <hardwareInterface>hardware_interface/VelocityJointInterface</hardwareInterface>
+    </joint>
+    <actuator name="Wheel_RL_motor">
+      <hardwareInterface>hardware_interface/VelocityJointInterface</hardwareInterface>
+      <mechanicalReduction>1</mechanicalReduction>
+    </actuator>
+  </transmission>
+  <!-- transmission -->
+  <link
+    name="Wheel_FR_Link">
+    <inertial>
+      <origin
+        xyz="-2.77555756156289E-16 -0.0241089810837368 7.7715611723761E-16"
+        rpy="0 0 0" />
+      <mass
+        value="5" />
+      <inertia
+        ixx="0.00350719044409909"
+        ixy="-4.35263549557573E-14"
+        ixz="7.08281671304654E-17"
+        iyy="0.00624534196811683"
+        iyz="-9.92550045529303E-14"
+        izz="0.00350719044409908" />
+    </inertial>
+    <visual>
+      <origin
+        xyz="0 0 0"
+        rpy="0 0 0" />
+      <geometry>
+        <mesh filename="file://${mesh_path}/Wheel_FR_Link.STL" />
+      </geometry>
+      <material
+        name="">
+        <color
+          rgba="0 0 0 1" />
+      </material>
+    </visual>
+    <collision>
+      <origin
+        xyz="0 0 0"
+        rpy="0 0 0" />
+      <geometry>
+        <mesh filename="file://${mesh_path}/Wheel_FR_Link.STL" />
+      </geometry>
+    </collision>
+  </link>
+  <joint
+    name="Wheel_FR_joint"
+    type="continuous">
+    <origin
+      xyz="0.545 -0.44 -0.747"
+      rpy="0 0 0" />
+    <parent
+      link="base_link" />
+    <child
+      link="Wheel_FR_Link" />
+    <axis
+      xyz="0 1 0" />
+  </joint>
+  <!-- transmission -->
+  <transmission name="Wheel_FR_trans">
+    <type>transmission_interface/SimpleTransmission</type>
+    <joint name="Wheel_FR_joint">
+      <hardwareInterface>hardware_interface/VelocityJointInterface</hardwareInterface>
+    </joint>
+    <actuator name="Wheel_FR_motor">
+      <hardwareInterface>hardware_interface/VelocityJointInterface</hardwareInterface>
+      <mechanicalReduction>1</mechanicalReduction>
+    </actuator>
+  </transmission>
+  <!-- transmission -->
+  <link
+    name="Wheel_RR_Link">
+    <inertial>
+      <origin
+        xyz="-1.22124532708767E-15 -0.0241089810837372 0"
+        rpy="0 0 0" />
+      <mass
+        value="5" />
+      <inertia
+        ixx="0.00350719044409917"
+        ixy="9.9248445809483E-14"
+        ixz="-6.92408075349762E-17"
+        iyy="0.00624534196811691"
+        iyz="-4.35245365048595E-14"
+        izz="0.00350719044409912" />
+    </inertial>
+    <visual>
+      <origin
+        xyz="0 0 0"
+        rpy="0 0 0" />
+      <geometry>
+        <mesh filename="file://${mesh_path}/Wheel_RR_Link.STL" />
+      </geometry>
+      <material
+        name="">
+        <color
+          rgba="0 0 0 1" />
+      </material>
+    </visual>
+    <collision>
+      <origin
+        xyz="0 0 0"
+        rpy="0 0 0" />
+      <geometry>
+        <mesh filename="file://${mesh_path}/Wheel_RR_Link.STL" />
+      </geometry>
+    </collision>
+  </link>
+  <joint
+    name="Wheel_RR_joint"
+    type="continuous">
+    <origin
+      xyz="-0.545 -0.44 -0.747"
+      rpy="0 0 0" />
+    <parent
+      link="base_link" />
+    <child
+      link="Wheel_RR_Link" />
+    <axis
+      xyz="0 1 0" />
+  </joint>
+  <!-- transmission -->
+  <transmission name="Wheel_RR_trans">
+    <type>transmission_interface/SimpleTransmission</type>
+    <joint name="Wheel_RR_joint">
+      <hardwareInterface>hardware_interface/VelocityJointInterface</hardwareInterface>
+    </joint>
+    <actuator name="Wheel_RR_motor">
+      <hardwareInterface>hardware_interface/VelocityJointInterface</hardwareInterface>
+      <mechanicalReduction>1</mechanicalReduction>
+    </actuator>
+  </transmission>
+  <!-- transmission -->
+  <gazebo reference="base_link">
+            <surface>
+                <friction>
+                    <ode>
+                        <mu>1</mu>
+                        <mu2>1</mu2>
+                        <slip1>0.1</slip1>
+                        <slip2>0</slip2>
+                        <fdir1>0 1 0</fdir1>
+                    </ode>
+                    <bullet>
+                        <friction>1</friction>
+                        <friction2>1</friction2>
+                        <rolling_friction>0.1</rolling_friction>
+                        <spinning_friction>0.1</spinning_friction>
+                    </bullet>
+                </friction>
+            </surface>
+        </gazebo>
+</robot>

File: install/robotpadi/share/robotpadi/urdf/ros2_control.xacro (robot description, xacro)
@@ -1 +1,33 @@
-/home/satyo03/TA_robotpadi/robotpadi/urdf/ros2_control.xacro
+<?xml version="1.0" encoding="utf-8"?>
+<robot xmlns:xacro="http://www.ros.org/wiki/xacro">
+  <ros2_control name="IgnitionSystem" type="system">
+    <hardware>
+      <plugin>gz_ros2_control/GazeboSimSystem</plugin>
+    </hardware>
+    <joint name="Wheel_FL_joint">
+      <command_interface name="velocity"/>
+      <state_interface name="position"/>
+      <state_interface name="velocity"/>
+    </joint>
+    <joint name="Wheel_RL_joint">
+      <command_interface name="velocity"/>
+      <state_interface name="position"/>
+      <state_interface name="velocity"/>
+    </joint>
+    <joint name="Wheel_FR_joint">
+      <command_interface name="velocity"/>
+      <state_interface name="position"/>
+      <state_interface name="velocity"/>
+    </joint>
+    <joint name="Wheel_RR_joint">
+      <command_interface name="velocity"/>
+      <state_interface name="position"/>
+      <state_interface name="velocity"/>
+    </joint>
+  </ros2_control>
+   <gazebo>
+      <plugin filename="gz_ros2_control-system" name="gz_ros2_control::GazeboSimROS2ControlPlugin">
+        <parameters>/home/satyo03/TA_robotpadi/install/robotpadi/share/robotpadi/config/diff_drive_controller.yaml</parameters>
+      </plugin>
+  </gazebo>
+</robot>

Commit message: ALHAMDULILLAH JALAN

File: install/robotpadi/share/robotpadi/urdf/gazebo_plugin.xacro (robot description, xacro)
@@ -13,5 +13,5 @@
   </gazebo> -->
   <gazebo>
-      <plugin filename="gz_ros2_control-system" name="gz_ros2_control::GazeboSimROS2ControlPlugin">
+      <plugin name="gz_ros2_control::GazeboSimROS2ControlPlugin" filename="libgz_ros2_control-system.so">
       <ros>
           <namespace>$(arg namespace)</namespace>

File: install/robotpadi/share/robotpadi/urdf/imu.xacro (robot description, xacro)
@@ -38,5 +38,18 @@
           <frame_id>${imu_link_name}</frame_id>
         </plugin> -->
-        <plugin filename="libgazebo_ros_imu_sensor.so" name="imu_plugin">
+        <sensor name="imu_sensor" type="imu">
+          <always_on>1</always_on>
+          <update_rate>100</update_rate>
+          <visualize>true</visualize>
+          <plugin name="gazebo_ros_imu_sensor" filename="libgazebo_ros_imu_sensor.so">
+            <ros>
+              <namespace>/</namespace>
+              <topic>/imu/data</topic>
+              <frame_id>base_link</frame_id>
+            </ros>
+            <initial_orientation_as_reference>false</initial_orientation_as_reference>
+          </plugin>
+        </sensor>
+        <!-- <plugin filename="libgazebo_ros_imu_sensor.so" name="imu_plugin">
           <ros>
             <namespace>/</namespace>
@@ -44,5 +57,5 @@
           </ros>
           <initial_orientation_as_reference>false</initial_orientation_as_reference>
-        </plugin>
+        </plugin> -->
       <!-- <imu>
         <angular_velocity>

File: install/robotpadi/share/robotpadi/urdf/robot_padi.xacro (robot description, xacro)
@@ -108,4 +108,16 @@
       xyz="0 1 0" />
   </joint>
+  <!-- blok biar berat -->
+  <gazebo reference="Wheel_FL_Link">
+    <mu1>1.0</mu1>
+    <mu2>1.0</mu2>
+    <kp>1000000.0</kp>
+    <kd>100.0</kd>
+    <minDepth>0.001</minDepth>
+    <maxVel>0.1</maxVel>
+    <fdir1>0 1 0</fdir1>
+    <material>Gazebo/Black</material>
+  </gazebo>
+<!-- blok biar berat -->
   <!-- transmission -->
   <transmission name="Wheel_FL_trans">
@@ -171,4 +183,16 @@
       xyz="0 1 0" />
   </joint>
+  <!-- blok biar berat -->
+  <gazebo reference="Wheel_RL_Link">
+    <mu1>1.0</mu1>
+    <mu2>1.0</mu2>
+    <kp>1000000.0</kp>
+    <kd>100.0</kd>
+    <minDepth>0.001</minDepth>
+    <maxVel>0.1</maxVel>
+    <fdir1>0 1 0</fdir1>
+    <material>Gazebo/Black</material>
+  </gazebo>
+<!-- blok biar berat -->
   <!-- transmission -->
   <transmission name="Wheel_RL_trans">
@@ -234,4 +258,16 @@
       xyz="0 1 0" />
   </joint>
+  <!-- blok biar berat -->
+  <gazebo reference="Wheel_FR_Link">
+    <mu1>1.0</mu1>
+    <mu2>1.0</mu2>
+    <kp>1000000.0</kp>
+    <kd>100.0</kd>
+    <minDepth>0.001</minDepth>
+    <maxVel>0.1</maxVel>
+    <fdir1>0 1 0</fdir1>
+    <material>Gazebo/Black</material>
+  </gazebo>
+<!-- blok biar berat -->
   <!-- transmission -->
   <transmission name="Wheel_FR_trans">
@@ -297,4 +333,16 @@
       xyz="0 1 0" />
   </joint>
+  <!-- blok biar berat -->
+  <gazebo reference="Wheel_RR_Link">
+    <mu1>1.0</mu1>
+    <mu2>1.0</mu2>
+    <kp>1000000.0</kp>
+    <kd>100.0</kd>
+    <minDepth>0.001</minDepth>
+    <maxVel>0.1</maxVel>
+    <fdir1>0 1 0</fdir1>
+    <material>Gazebo/Black</material>
+  </gazebo>
+<!-- blok biar berat -->
   <!-- transmission -->
   <transmission name="Wheel_RR_trans">
@@ -309,4 +357,13 @@
   </transmission>
   <!-- transmission -->
+  <plugin name="gazebo_ros_odometry" filename="libgazebo_ros_odometry.so">
+    <ros>
+      <robotNamespace>/robotpadi</robotNamespace>
+      <topicName>/odom</topicName>
+    </ros>
+    <publish_odom>true</publish_odom>
+    <publish_tf>true</publish_tf>
+    ...
+  </plugin>
   <gazebo reference="base_link">
             <surface>
@@ -327,4 +384,4 @@
                 </friction>
             </surface>
-        </gazebo>
+  </gazebo>
 </robot>
