Commit message: add imu and modify robotpadi.xacro and launch

File: robotpadi/urdf/main.xacro (robot description, xacro)
@@ -3,4 +3,5 @@
     <xacro:include filename="robot_padi.xacro"/>
     <xacro:include filename="ros2_control.xacro"/>
+    <xacro:include filename="imu.xacro"/>
     <!-- <xacro:include filename="gazebo_plugin.xacro"/> -->
 </robot>

File: robotpadi/urdf/robot_padi.xacro (robot description, xacro)
@@ -5,4 +5,5 @@
 <robot xmlns:xacro="http://www.ros.org/wiki/xacro">
   <xacro:property name="mesh_path" value="$(find robotpadi)/meshes"/>
+  <xacro:include filename="$(find robotpadi)/urdf/imu.xacro" />
   <link name="base_footprint"/>
   <joint name="base_footprint_to_base_link_joint" type="fixed">
@@ -17,6 +18,6 @@
         rpy="0 0 0" />
       <mass
-        value="49.9119470217901" />
-      <inertia
+        value="180" />
+      <!-- <inertia
         ixx="2.32881913674761"
         ixy="3.13125017353562E-06"
@@ -24,5 +25,12 @@
         iyy="1.87881391838459"
         iyz="-1.67327823321756E-07"
-        izz="2.97314088623897" />
+        izz="2.97314088623897" /> -->
+      <inertia
+        ixx="25.4"
+        ixy="0"
+        ixz="0"
+        iyy="35.1"
+        iyz="0"
+        izz="38.2" />
     </inertial>
     <visual>
@@ -36,5 +44,5 @@
         name="">
         <color
-          rgba="0.792156862745098 0.819607843137255 0.933333333333333 1" />
+          rgba="0 0 1 1" />
       </material>
     </visual>
@@ -48,4 +56,5 @@
     </collision>
   </link>
+   <xacro:imu_sensor parent_link="base_link" imu_link_name="imu_link" origin_xyz="0 0 0.05" origin_rpy="0 0 0"/>
   <link
     name="Wheel_FL_Link">
@@ -55,5 +64,5 @@
         rpy="0 0 0" />
       <mass
-        value="0.378233531013503" />
+        value="5" />
       <inertia
         ixx="0.00350719044409918"
@@ -74,5 +83,5 @@
         name="">
         <color
-          rgba="0.109803921568627 0.109803921568627 0.109803921568627 1" />
+          rgba="0 0 0 1" />
       </material>
     </visual>
@@ -106,5 +115,5 @@
         rpy="0 0 0" />
       <mass
-        value="0.378233531013499" />
+        value="5" />
       <inertia
         ixx="0.00350719044409904"
@@ -125,5 +134,5 @@
         name="">
         <color
-          rgba="0.109803921568627 0.109803921568627 0.109803921568627 1" />
+          rgba="0 0 0 1" />
       </material>
     </visual>
@@ -157,5 +166,5 @@
         rpy="0 0 0" />
       <mass
-        value="0.378233531013493" />
+        value="5" />
       <inertia
         ixx="0.00350719044409909"
@@ -176,5 +185,5 @@
         name="">
         <color
-          rgba="0.109803921568627 0.109803921568627 0.109803921568627 1" />
+          rgba="0 0 0 1" />
       </material>
     </visual>
@@ -199,5 +208,5 @@
       link="Wheel_FR_Link" />
     <axis
-      xyz="0 -1 0" />
+      xyz="0 1 0" />
   </joint>
   <link
@@ -208,5 +217,5 @@
         rpy="0 0 0" />
       <mass
-        value="0.37823353101351" />
+        value="5" />
       <inertia
         ixx="0.00350719044409917"
@@ -227,5 +236,5 @@
         name="">
         <color
-          rgba="0.109803921568627 0.109803921568627 0.109803921568627 1" />
+          rgba="0 0 0 1" />
       </material>
     </visual>
@@ -250,5 +259,24 @@
       link="Wheel_RR_Link" />
     <axis
-      xyz="0 -1 0" />
-  </joint>
+      xyz="0 1 0" />
+  </joint>
+  <gazebo reference="base_link">
+            <surface>
+                <friction>
+                    <ode>
+                        <mu>1</mu>
+                        <mu2>1</mu2>
+                        <slip1>0.1</slip1>
+                        <slip2>0</slip2>
+                        <fdir1>0 1 0</fdir1>
+                    </ode>
+                    <bullet>
+                        <friction>1</friction>
+                        <friction2>1</friction2>
+                        <rolling_friction>0.1</rolling_friction>
+                        <spinning_friction>0.1</spinning_friction>
+                    </bullet>
+                </friction>
+            </surface>
+        </gazebo>
 </robot>
