Commit message: baru smc

File: robotpadi/urdf/robot_padi.xacro (robot description, xacro)
@@ -108,4 +108,16 @@
       xyz="0 1 0" />
   </joint>
+  <!-- transmission -->
+  <transmission name="Wheel_FL_trans">
+    <type>transmission_interface/SimpleTransmission</type>
+    <joint name="Wheel_FL_joint">
+      <hardwareInterface>hardware_interface/VelocityJointInterface</hardwareInterface>
+    </joint>
+    <actuator name="Wheel_FL_motor">
+      <hardwareInterface>hardware_interface/VelocityJointInterface</hardwareInterface>
+      <mechanicalReduction>1</mechanicalReduction>
+    </actuator>
+  </transmission>
+<!-- transmission -->
   <link
     name="Wheel_RL_Link">
@@ -159,4 +171,16 @@
       xyz="0 1 0" />
   </joint>
+  <!-- transmission -->
+  <transmission name="Wheel_RL_trans">
+    <type>transmission_interface/SimpleTransmission</type>
+    <joint name="Wheel_RL_joint">
+      <hardwareInterface>hardware_interface/VelocityJointInterface</hardwareInterface>
+    </joint>
+    <actuator name="Wheel_RL_motor">
+      <hardwareInterface>hardware_interface/VelocityJointInterface</hardwareInterface>
+      <mechanicalReduction>1</mechanicalReduction>
+    </actuator>
+  </transmission>
+  <!-- transmission -->
   <link
     name="Wheel_FR_Link">
@@ -210,4 +234,16 @@
       xyz="0 1 0" />
   </joint>
+  <!-- transmission -->
+  <transmission name="Wheel_FR_trans">
+    <type>transmission_interface/SimpleTransmission</type>
+    <joint name="Wheel_FR_joint">
+      <hardwareInterface>hardware_interface/VelocityJointInterface</hardwareInterface>
+    </joint>
+    <actuator name="Wheel_FR_motor">
+      <hardwareInterface>hardware_interface/VelocityJointInterface</hardwareInterface>
+      <mechanicalReduction>1</mechanicalReduction>
+    </actuator>
+  </transmission>
+  <!-- transmission -->
   <link
     name="Wheel_RR_Link">
@@ -261,4 +297,16 @@
       xyz="0 1 0" />
   </joint>
+  <!-- transmission -->
+  <transmission name="Wheel_RR_trans">
+    <type>transmission_interface/SimpleTransmission</type>
+    <joint name="Wheel_RR_joint">
+      <hardwareInterface>hardware_interface/VelocityJointInterface</hardwareInterface>
+    </joint>
+    <actuator name="Wheel_RR_motor">
+      <hardwareInterface>hardware_interface/VelocityJointInterface</hardwareInterface>
+      <mechanicalReduction>1</mechanicalReduction>
+    </actuator>
+  </transmission>
+  <!-- transmission -->
   <gazebo reference="base_link">
             <surface>
